Commit message: Updated scanbot urdf description to include transmissions and plugin

File: docker/ros-files/scanbot.urdf (robot description, URDF)
Before this commit: robot scanbot, 4 links, 3 joints
Links:
- removed link scanbot__chassis
- removed link scanbot__left_wheel
- removed link scanbot__right_wheel
- removed link scanbot__tower
- added link scanbot_chassis, mass 0.5; collision box size=0.160 0.100 0.065; collision sphere radius=0.02
- added link scanbot_left_wheel, mass 0.075; collision cylinder length=0.018 radius=0.03; visual cylinder length=0.018 radius=0.03
- added link scanbot_right_wheel, mass 0.075; collision cylinder length=0.018 radius=0.03; visual cylinder length=0.018 radius=0.03
- added link scanbot_tower, mass 0.050; collision cylinder length=0.06 radius=0.02; visual cylinder length=0.06 radius=0.02
Joints:
- removed joint scanbot__left_wheel_revolute
- removed joint scanbot__right_wheel_revolute
- removed joint scanbot__tower_revolute
- added joint scanbot_left_wheel_revolute: type continuous, parent scanbot_chassis, child scanbot_left_wheel, origin xyz=0 0.05 0.02749 rpy=0 1.5707 1.5707, axis 0 0 1, limit effort=80 velocity=25.1327412287
- added joint scanbot_right_wheel_revolute: type continuous, parent scanbot_chassis, child scanbot_right_wheel, origin xyz=0 -0.05 0.0275 rpy=0 1.5707 1.5707, axis 0 0 1, limit effort=80 velocity=25.1327412287
- added joint scanbot_tower_revolute: type revolute, parent scanbot_chassis, child scanbot_tower, origin xyz=-0.01 0 0.083 rpy=0 0 0, axis 0 0 1, limit lower=0 upper=0 effort=0 velocity=0

Commit message: Renamed robot base in urdf file and added a sensor

File: docker/ros-files/scanbot.urdf (robot description, URDF)
Before this commit: robot scanbot, 4 links, 3 joints
Links:
- removed link scanbot_chassis
- added link base_link, mass 0.5; collision box size=0.160 0.100 0.065; collision sphere radius=0.02
Joints:
- joint scanbot_left_wheel_revolute: parent scanbot_chassis -> base_link
- joint scanbot_right_wheel_revolute: parent scanbot_chassis -> base_link
- joint scanbot_tower_revolute: parent scanbot_chassis -> base_link

Commit message: Trimmed values to properly represent robots odometry and scans

File: docker/ros-files/scanbot.urdf (robot description, URDF)
Before this commit: robot scanbot, 4 links, 3 joints
Joints:
- joint scanbot_left_wheel_revolute: limit effort=80 velocity=25.1327412287 -> effort=100 velocity=3.33
- joint scanbot_right_wheel_revolute: limit effort=80 velocity=25.1327412287 -> effort=100 velocity=3.33
